Commit message: xacro gazebo changes

File: src/my_robot/urdf/my_robot.xacro (robot description, xacro)
@@ -11,5 +11,5 @@
 <joint name="camera_optical_joint" type="fixed">
     <origin xyz="0 0 0" rpy="-1.5707 0 -1.5707"/>
-    <parent link="camera_link"/>
+    <parent link="camera"/>
     <child link="camera_link_optical"/>
   </joint>
